File: kicad/roverProject.kicad_sch (KiCad schematic)
At the start: 7 parts, among them M1 DC Motor w/ Encoder, M2 DC Motor w/ Encoder

Commit message: Create motor-control.cpp
Will add description later!
Parts:
- added U1: MPU-6050, Sensor_Motion:InvenSense_QFN-24_4x4mm_P0.5mm, symbol Sensor_Motion:MPU-6050
Connections:
- net +5V: now also U1.13 (VDD), U1.8 (VLOGIC)
- net GND: now also U1.18 (GND)
- net SDA_3V3: now reaches A1.31 (SDA/A4)
- net SDA_3V3: now also U1.24 (SDA)
- net SCL_3V3: now reaches A1.32 (SCL/A5)
- net SCL_3V3: now also U1.23 (SCL)
Other:
- moved on the sheet: BZ1
